Commit message: tt

File: panda_coarse/panda_7link.urdf (robot description, URDF)
Before this commit: robot panda, 14 links, 13 joints
Joints:
- joint world_joint: origin xyz=1.0 1.0 0.85 rpy=0.0 0.0 0.0 -> xyz=0.4 0.6 0 rpy=0.0 0.0 0.0

Commit message: dd

File: panda_coarse/panda_7link.urdf (robot description, URDF)
Before this commit: robot panda, 14 links, 13 joints
Links:
- link panda_hand: geometry collision mesh filename=meshes/collision/hand.obj; visual mesh filename=meshes/visual/hand.stl
- link panda_leftfinger: geometry collision mesh filename=meshes/collision/finger.obj; visual mesh filename=meshes/visual/finger.stl
- link panda_link0: geometry collision mesh filename=meshes/collision/link0.obj; visual mesh filename=meshes/visual/link0.stl
- link panda_link1: geometry collision mesh filename=meshes/collision/link1.obj; visual mesh filename=meshes/visual/link1.stl
- link panda_link2: geometry collision mesh filename=meshes/collision/link2.obj; visual mesh filename=meshes/visual/link2.stl
- link panda_link3: geometry collision mesh filename=meshes/collision/link3.obj; visual mesh filename=meshes/visual/link3.stl
- link panda_link4: geometry collision mesh filename=meshes/collision/link4.obj; visual mesh filename=meshes/visual/link4.stl
- link panda_link5: geometry collision mesh filename=meshes/collision/link5.obj; visual mesh filename=meshes/visual/link5.stl
- link panda_link6: geometry collision mesh filename=meshes/collision/link6.obj; visual mesh filename=meshes/visual/link6.stl
- link panda_link7: geometry collision mesh filename=meshes/collision/link7.obj; visual mesh filename=meshes/visual/link7.stl
- link panda_rightfinger: geometry collision mesh filename=meshes/collision/finger.obj; visual mesh filename=meshes/visual/finger.stl
Joints:
- joint world_joint: origin xyz=0.4 0.6 0 rpy=0.0 0.0 0.0 -> xyz=0.5 0.5 0.0 rpy=0.0 0.0 0.0

Commit message: dd

File: panda_coarse/panda_7link.urdf (robot description, URDF)
Before this commit: robot panda, 14 links, 13 joints
Joints:
- joint world_joint: origin xyz=0.5 0.5 0.0 rpy=0.0 0.0 0.0 -> xyz=2.0 2.0 0.5 rpy=0.0 0.0 0.0

File: panda_coarse_collision/panda_7link_collision.urdf (robot description, URDF)
Before this commit: robot panda_col, 14 links, 13 joints
Joints:
- joint world_joint: origin xyz=0.5 0.5 0.0 rpy=0.0 0.0 0.0 -> xyz=2.0 2.0 0.5 rpy=0.0 0.0 0.0
